File: src/audiocardio.kicad_pcb (KiCad board)
At the start: 2 copper layers, 47.1 x 72.1 mm, 42 parts, among them J1 USB_A, J2 AudioJack3, J4 AudioJack3, U1 PCM2912APJTR, Y1 6MHz

Commit message: Changes
Parts:
- removed J1: USB_A, Connector_USB:USB_A_Connfly_DS1098_Horizontal
- added J2: USB_A_PLUG, connectors:usb-PCB, F.Cu at (137.0, 118.3)
Routing:
- net /P: track 21.6 -> 34.7 mm
- net /N: track 22.0 -> 34.6 mm
- net VBUS: track 42.2 -> 54.8 mm
Other:
- board size 47.1 x 72.1 mm -> 47.1 x 84.1 mm

Commit message: changing stuff
Parts:
- removed D1, D2: LED, LED_SMD:LED_0603_1608Metric
- removed the J2 at (137.0, 118.3)
- removed R10, R11: 3.3k, Resistor_SMD:R_0603_1608Metric
- C7: footprint Capacitor_SMD:C_0603_1608Metric -> Capacitor_THT:C_Radial_D4.0mm_H5.0mm_P1.50mm
- R1, R2, R3, R4, R5, R8, R9: footprint Resistor_SMD:R_0603_1608Metric -> Resistor_THT:R_Axial_DIN0204_L3.6mm_D1.6mm_P5.08mm_Horizontal
- moved G*** 36.9 mm to (125.6, 94.3)
- moved G*** 32.8 mm to (151.3, 66.9)
- moved G*** 16.6 mm to (121.9, 76.9), turned to 90 degrees
- moved C14 9.59 mm to (124.2, 57.3)
- moved R8 8.81 mm to (153.2, 81.2)
- moved R9 6.44 mm to (128.3, 58.5)
- moved R5 6.13 mm to (153.3, 59.6)
- moved R3 5.99 mm to (135.1, 54.3), turned to 90 degrees
- moved C7 5.16 mm to (149.9, 76.4), turned to 90 degrees
- moved R1 3.87 mm to (139.8, 83.0)
- moved R4 3.57 mm to (149.1, 49.2), turned to -90 degrees
- moved R2 3.49 mm to (137.6, 61.0)
- moved C4 1.50 mm to (136.1, 82.2)
Routing:
- net VBUS: track 54.8 -> 40.7 mm
- net GND: track 28.8 -> 41.5 mm
- net XT+: track 28.2 -> 36.2 mm
- net /N: track 34.6 -> 42.5 mm
- net VCOM1: track 4.80 -> 10.5 mm
- net XT-: track 20.3 -> 25.6 mm
- net /P: track 34.7 -> 39.0 mm
- net PLAY: track 3.79 -> 0.00 mm
- net Net-(C13-Pad2): track 12.1 -> 15.8 mm
- net REC: track 3.47 -> 0.17 mm
- net Net-(C12-Pad2): track 12.0 -> 15.3 mm
- net VDD: track 5.85 -> 8.75 mm
- net MicIn: track 23.4 -> 21.6 mm
- net VOUTR: track 22.8 -> 24.3 mm
- net Net-(D2-K): track 1.46 -> 0.00 mm
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Other:
- board size 47.1 x 84.1 mm -> 47.1 x 85.5 mm
