File: src/audiocardio.kicad_sch (KiCad schematic)
At the start: 35 parts, among them J1 USB_A, J2 AudioJack3, J4 AudioJack3, U1 PCM2912APJTR, Y1 6MHz

Commit message: changing stuff
Parts:
- removed D1, D2: LED, LED_SMD:LED_0603_1608Metric, symbol Device:LED
- removed R10, R11: 3.3k, Resistor_SMD:R_0603_1608Metric, symbol Device:R
- C7: footprint Capacitor_SMD:C_0603_1608Metric -> Capacitor_THT:C_Radial_D4.0mm_H5.0mm_P1.50mm
- R1, R2, R3, R4, R5, R8, R9: footprint Resistor_SMD:R_0603_1608Metric -> Resistor_THT:R_Axial_DIN0204_L3.6mm_D1.6mm_P5.08mm_Horizontal
